Commit message: moving more prefabs to the correct location

File: Runtime/Prefabs/ur5e/ur5e.urdf (robot description, URDF)
Before this commit: robot ur, 13 links, 12 joints
Links:
- removed link ft_frame
- link base_link_inertia: geometry collision mesh filename=package://ur_description/meshes/ur5e/collision/base.stl; visual mesh filename=package://ur_description/meshes/ur5e/visual/base.dae
- link forearm_link: geometry collision mesh filename=package://ur_description/meshes/ur5e/collision/forearm.stl; visual mesh filename=package://ur_description/meshes/ur5e/visual/forearm.dae
- link shoulder_link: geometry collision mesh filename=package://ur_description/meshes/ur5e/collision/shoulder.stl; visual mesh filename=package://ur_description/meshes/ur5e/visual/shoulder.dae
- link upper_arm_link: geometry collision mesh filename=package://ur_description/meshes/ur5e/collision/upperarm.stl; visual mesh filename=package://ur_description/meshes/ur5e/visual/upperarm.dae
- link wrist_1_link: geometry collision mesh filename=package://ur_description/meshes/ur5e/collision/wrist1.stl; visual mesh filename=package://ur_description/meshes/ur5e/visual/wrist1.dae
- link wrist_2_link: geometry collision mesh filename=package://ur_description/meshes/ur5e/collision/wrist2.stl; visual mesh filename=package://ur_description/meshes/ur5e/visual/wrist2.dae
- link wrist_3_link: geometry collision mesh filename=package://ur_description/meshes/ur5e/collision/wrist3.stl; visual mesh filename=package://ur_description/meshes/ur5e/visual/wrist3.dae
Joints:
- removed joint base_joint
- removed joint wrist_3_link-ft_frame
- added joint joint_world: type fixed, parent world, child base_link, origin xyz=0 0 0 rpy=0 0 0
